File: RPi Voltage Regulator Board/RPi Voltage Regulator Board.kicad_pcb (KiCad board)
At the start: 2 copper layers, 21.6 x 24.1 mm, 20 parts, among them J3 CONN_01X02, J4 CONN_01X02, J5 CONN_01X02, J6 PWM, J7 PWM, J8 PWM, Q1 PN2222, Q2 PN2222, Q3 PN2222, U1 AMS1117-5.0

Commit message: Board rev 1.1
Parts:
- removed J3, J4, J5: CONN_01X02, Pin_Headers:Pin_Header_Straight_1x02
- removed J6, J7, J8: PWM, Pin_Headers:Pin_Header_Straight_1x03
- removed Pi: RPI Header 4-10, Pin_Headers:Pin_Header_Straight_1x04_Pitch2.54mm
- removed Q1, Q2, Q3: PN2222, TO_SOT_Packages_THT:TO-92_Inline_Narrow_Oval
- removed R1, R2, R3: 10k, Resistors_SMD:R_0805_HandSoldering
- removed R4: 29, Resistors_THT:R_Axial_DIN0516_L15.5mm_D5.0mm_P7.62mm_Vertical
- removed R5, R6: 17, Resistors_THT:R_Axial_DIN0516_L15.5mm_D5.0mm_P7.62mm_Vertical
- added J1: RPi 4-12, Pin_Headers:Pin_Header_Straight_1x05, F.Cu at (140.7, 107.5)
- added P0: CONN_01X02, Pin_Headers:Pin_Header_Straight_1x02, F.Cu at (200.9, 124.1)
- added P0: PWM, Pin_Headers:Pin_Header_Straight_1x03, F.Cu at (197.8, 105.6)
- added P0: CONN_01X02, Pin_Headers:Pin_Header_Straight_1x02, F.Cu at (164.8, 124.1)
- added P0: PWM, Pin_Headers:Pin_Header_Straight_1x03, F.Cu at (168.6, 100.5)
- added P1: CONN_01X02, Pin_Headers:Pin_Header_Straight_1x02, F.Cu at (194.8, 124.1)
- added P1: PWM, Pin_Headers:Pin_Header_Straight_1x03, F.Cu at (195.3, 105.6)
- added P1: CONN_01X02, Pin_Headers:Pin_Header_Straight_1x02, F.Cu at (170.7, 124.1)
- added P1: PWM, Pin_Headers:Pin_Header_Straight_1x03, F.Cu at (171.2, 100.5)
- added P2: PWM, Pin_Headers:Pin_Header_Straight_1x03, F.Cu at (192.8, 105.6)
- added P2: CONN_01X02, Pin_Headers:Pin_Header_Straight_1x02, F.Cu at (189.0, 124.1)
- added P2: CONN_01X02, Pin_Headers:Pin_Header_Straight_1x02, F.Cu at (176.8, 124.1)
- added P2: PWM, Pin_Headers:Pin_Header_Straight_1x03, F.Cu at (173.7, 100.5)
- added Q4: MMBT2222, TO_SOT_Packages_SMD:SOT-23_Handsoldering, F.Cu at (190.5, 118.5)
- added Q4: MMBT2222, TO_SOT_Packages_SMD:SOT-23_Handsoldering, F.Cu at (166.4, 118.5)
- added Q5: MMBT2222, TO_SOT_Packages_SMD:SOT-23_Handsoldering, F.Cu at (196.0, 118.5)
- added Q5: MMBT2222, TO_SOT_Packages_SMD:SOT-23_Handsoldering, F.Cu at (171.9, 118.5)
- added Q6: MMBT2222, TO_SOT_Packages_SMD:SOT-23_Handsoldering, F.Cu at (200.7, 118.5)
- added Q6: MMBT2222, TO_SOT_Packages_SMD:SOT-23_Handsoldering, F.Cu at (176.6, 118.5)
- added R10: 10k, Resistors_SMD:R_1206_HandSoldering, F.Cu at (190.2, 111.4)
- added R10: 10k, Resistors_SMD:R_1206_HandSoldering, F.Cu at (166.1, 111.4)
- added R11: 10k, Resistors_SMD:R_1206_HandSoldering, F.Cu at (195.8, 111.4)
- added R11: 10k, Resistors_SMD:R_1206_HandSoldering, F.Cu at (171.7, 111.4)
- added R12: 10k, Resistors_SMD:R_1206_HandSoldering, F.Cu at (201.4, 111.4)
- added R12: 10k, Resistors_SMD:R_1206_HandSoldering, F.Cu at (177.3, 111.4)
- added R7: 29, Resistors_THT:R_Axial_DIN0516_L15.5mm_D5.0mm_P7.62mm_Vertical, F.Cu at (190.2, 129.7)
- added R7: 29, Resistors_THT:R_Axial_DIN0516_L15.5mm_D5.0mm_P7.62mm_Vertical, F.Cu at (166.1, 129.7)
- added R8: 29, Resistors_THT:R_Axial_DIN0516_L15.5mm_D5.0mm_P7.62mm_Vertical, F.Cu at (196.3, 129.7)
- added R8: 29, Resistors_THT:R_Axial_DIN0516_L15.5mm_D5.0mm_P7.62mm_Vertical, F.Cu at (172.2, 129.7)
- added R9: 29, Resistors_THT:R_Axial_DIN0516_L15.5mm_D5.0mm_P7.62mm_Vertical, F.Cu at (202.4, 129.7)
- added R9: 29, Resistors_THT:R_Axial_DIN0516_L15.5mm_D5.0mm_P7.62mm_Vertical, F.Cu at (178.3, 129.7)
- added SDWN1: TAC_SWITCH_6x6mm, SpadeConnector:TacButton_6mm_6mm, F.Cu at (148.9, 121.4)
Connections:
- Nodes pad 1: Net-(J1-Pad1) -> (no net)
- Nodes pad 2: Net-(J1-Pad2) -> (no net)
- U1 pad 3: Net-(J1-Pad2) -> Net-(Nodes1-Pad2)
Routing:
- net Net-(J13-Pad1): track 0.00 -> 20.6 mm
- net Net-(J14-Pad1): track 0.00 -> 17.4 mm, vias 0 -> 1
- net Net-(J1-Pad3): track 0.00 -> 17.3 mm
- net Net-(J1-Pad1): track 17.3 -> 0.00 mm
- net Net-(J12-Pad1): track 0.00 -> 15.0 mm
- net Net-(J11-Pad1): track 0.00 -> 12.4 mm
- net Net-(J10-Pad1): track 0.00 -> 12.4 mm
- net Net-(J9-Pad1): track 0.00 -> 12.2 mm
- net Net-(J11-Pad2): track 0.00 -> 10.5 mm
- net Net-(J10-Pad2): track 0.00 -> 10.2 mm
- net Net-(J9-Pad2): track 0.00 -> 9.95 mm
- net Net-(Q4-Pad1): track 0.00 -> 9.58 mm
- net Net-(Q5-Pad1): track 0.00 -> 9.52 mm
- net Net-(Nodes1-Pad2): track 0.00 -> 7.84 mm
- net Net-(J1-Pad2): track 7.84 -> 0.00 mm
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- added copper zone on B.Cu, net +5V
- added copper zone on F.Cu, net GND
Other:
- board size 21.6 x 24.1 mm -> 69.8 x 45.7 mm
- net class Power added: clearance 0.3, trace_width 0.4, via_dia 0.6, via_drill 0.4
- board text added: "PWM Adapter"
