File: RPi Voltage Regulator Board/RPi Voltage Regulator Board.sch (KiCad schematic (older format))
At the start: 20 parts, among them J1 Node Bus, J2 RPI Header 4-10, J3 CONN_01X02, J4 CONN_01X02, J5 CONN_01X02, J6 PWM, J7 PWM, J8 PWM, Q1 PN2222, Q2 PN2222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

Commit message: Board rev 1.1
Parts:
- removed J2: RPI Header 4-10, Pin_Headers:Pin_Header_Straight_1x04_Pitch2.54mm, symbol CONN_01X04
- removed J3, J4, J5: CONN_01X02, Pin_Headers:Pin_Header_Straight_1x02, symbol CONN_01X02
- removed J6, J7, J8: PWM, Pin_Headers:Pin_Header_Straight_1x03, symbol CONN_01X03
- removed Q1, Q2, Q3: PN2222, TO_SOT_Packages_THT:TO-92_Inline_Narrow_Oval, symbol PN2222
- removed R1, R2, R3: 10k, Resistors_SMD:R_0805_HandSoldering, symbol R
- removed R4: 29, Resistors_THT:R_Axial_DIN0516_L15.5mm_D5.0mm_P7.62mm_Vertical, symbol R
- removed R5, R6: 17, Resistors_THT:R_Axial_DIN0516_L15.5mm_D5.0mm_P7.62mm_Vertical, symbol R
- added J1: RPi 4-12, Pin_Headers:Pin_Header_Straight_1x05, symbol CONN_01X05
- added J10, J11, J9: CONN_01X02, Pin_Headers:Pin_Header_Straight_1x02, symbol CONN_01X02
- added J12, J13, J14: PWM, Pin_Headers:Pin_Header_Straight_1x03, symbol CONN_01X03
- added Q4, Q5, Q6: MMBT2222, TO_SOT_Packages_SMD:SOT-23_Handsoldering, symbol MMBT2222
- added R10, R11, R12: 10k, Resistors_SMD:R_1206_HandSoldering, symbol R
- added R7, R8, R9: 29, Resistors_THT:R_Axial_DIN0516_L15.5mm_D5.0mm_P7.62mm_Vertical, symbol R
- added SDWN1: TAC_SWITCH_6x6mm, SpadeConnector:TacButton_6mm_6mm, symbol TAC_SWITCH_6x6mm
- renumbered J1 to Nodes1
Connections:
- net +5V: now also J12.2 (P2), J13.2 (P2), J14.2 (P2), R7.2, R8.2, R9.2
- net GND: now also J12.3 (P3), J13.3 (P3), J14.3 (P3), Q4.2 (E), Q5.2 (E), Q6.2 (E)
- net at C1.1, C2.1, U1.2 (VO)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: now also J1.1 (P1)
- net at C1.2, C2.2, Nodes1.3 (P3)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: now also J1.2 (P2), SDWN1.2
- net at Nodes1.1 (P1): now also J1.3 (P3)
- net at Nodes1.4 (P4): now also J1.4 (P4)
- new net: J12.1 (P1), R10.2
- new net: J9.1 (P1), R7.1
- new net: J9.2 (P2), Q4.3 (C)
- new net: Q4.1 (B), R10.1
- new net: J13.1 (P1), R11.2
- new net: J10.1 (P1), R8.1
- new net: J10.2 (P2), Q5.3 (C)
- new net: Q5.1 (B), R11.1
- new net: J14.1 (P1), R12.2
- new net: J11.1 (P1), R9.1
- new net: J11.2 (P2), Q6.3 (C)
- new net: Q6.1 (B), R12.1
- new net: J1.5 (P5), SDWN1.1
- no-connect marks 0 -> 2
